File: HW/KiCAD/AnalogSumm2CH.kicad_sch (KiCad schematic)
At the start: 24 parts, among them U41 NE5532, U45 NE5532

Commit message: some eidts, remove com
Parts:
- renumbered C203 to C194, C204 to C195, C205 to C196, C206 to C197, L24 to L23, L25 to L24, R186 to R173, R187 to R174, R192 to R175, R193 to R176, R188 to R177, R189 to R178, R195 to R179, R190 to R180, R194 to R181, R191 to R182, R196 to R183, R197 to R184, R198 to R185, R199 to R186, R200 to R187, R201 to R188, U41 to U35, U45 to U36, U41 to U37
Changed lines of the file:
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@@
 		(dnp no)
 		(fields_autoplaced yes)
-		(property "Reference" "L24"
+		(property "Reference" "L23"
 			(at 35.56 40.64 90)
 			(effects
@@
 			(project "kharon386mod_by_maxssau"
 				(path "/48e19dd7-3c62-4fd7-8a3b-78a40c79d086/523f9a2f-ddd1-4c6e-b1cf-fbf0997bf88b/7af472cf-3fd2-4e4b-b7f3-feb3f131a7f1"
-					(reference "L24")
+					(reference "L23")
 					(unit 1)
 				)
@@
 		(dnp no)
 		(fields_autoplaced yes)
-		(property "Reference" "R188"
+		(property "Reference" "R177"
 			(at 58.42 39.37 90)
 			(effects
@@
 			(project "kharon386mod_by_maxssau"
 				(path "/48e19dd7-3c62-4fd7-8a3b-78a40c79d086/523f9a2f-ddd1-4c6e-b1cf-fbf0997bf88b/7af472cf-3fd2-4e4b-b7f3-feb3f131a7f1"
-					(reference "R188")
+					(reference "R177")
 					(unit 1)
 				)
@@
 		(dnp no)
 		(fields_autoplaced yes)
-		(property "Reference" "R193"
+		(property "Reference" "R176"
 			(at 45.72 105.41 90)
 			(effects
@@
 			(project "kharon386mod_by_maxssau"
 				(path "/48e19dd7-3c62-4fd7-8a3b-78a40c79d086/523f9a2f-ddd1-4c6e-b1cf-fbf0997bf88b/7af472cf-3fd2-4e4b-b7f3-feb3f131a7f1"
-					(reference "R193")
+					(reference "R176")
 					(unit 1)
 				)
@@
 		(on_board yes)
 		(dnp no)
-		(property "Reference" "U45"
+		(property "Reference" "U36"
 			(at 207.0101 111.76 90)
 			(effects
@@
 			(project ""
 				(path "/48e19dd7-3c62-4fd7-8a3b-78a40c79d086/523f9a2f-ddd1-4c6e-b1cf-fbf0997bf88b/7af472cf-3fd2-4e4b-b7f3-feb3f131a7f1"
-					(reference "U45")
+					(reference "U36")
 					(unit 2)
 				)
@@
 		(dnp no)
 		(fields_autoplaced yes)
-		(property "Reference" "C203"
+		(property "Reference" "C194"
 			(at 49.53 48.2599 0)
 			(effects
@@
 			(project "kharon386mod_by_maxssau"
 				(path "/48e19dd7-3c62-4fd7-8a3b-78a40c79d086/523f9a2f-ddd1-4c6e-b1cf-fbf0997bf88b/7af472cf-3fd2-4e4b-b7f3-feb3f131a7f1"
-					(reference "C203")
+					(reference "C194")
 					(unit 1)
 				)
@@
 		(dnp no)
 		(fields_autoplaced yes)
-		(property "Reference" "R198"
+		(property "Reference" "R185"
 			(at 189.23 129.54 90)
 			(effects
@@
 			(project "kharon386mod_by_maxssau"
 				(path "/48e19dd7-3c62-4fd7-8a3b-78a40c79d086/523f9a2f-ddd1-4c6e-b1cf-fbf0997bf88b/7af472cf-3fd2-4e4b-b7f3-feb3f131a7f1"
-					(reference "R198")
+					(reference "R185")
 					(unit 1)
 				)
@@
 		(dnp no)
 		(fields_autoplaced yes)
-		(property "Reference" "R186"
+		(property "Reference" "R173"
 			(at 35.56 46.99 90)
 			(effects
@@
 			(project "kharon386mod_by_maxssau"
 				(path "/48e19dd7-3c62-4fd7-8a3b-78a40c79d086/523f9a2f-ddd1-4c6e-b1cf-fbf0997bf88b/7af472cf-3fd2-4e4b-b7f3-feb3f131a7f1"
-					(reference "R186")
+					(reference "R173")
 					(unit 1)
 				)
@@
 		(dnp no)
 		(fields_autoplaced yes)
-		(property "Reference" "R195"
+		(property "Reference" "R179"
 			(at 68.58 132.08 90)
 			(effects
@@
 			(project "kharon386mod_by_maxssau"
 				(path "/48e19dd7-3c62-4fd7-8a3b-78a40c79d086/523f9a2f-ddd1-4c6e-b1cf-fbf0997bf88b/7af472cf-3fd2-4e4b-b7f3-feb3f131a7f1"
-					(reference "R195")
+					(reference "R179")
 					(unit 1)
 				)
@@
 		(dnp no)
 		(fields_autoplaced yes)
-		(property "Reference" "R200"
+		(property "Reference" "R187"
 			(at 205.74 129.54 90)
 			(effects
@@
 			(project "kharon386mod_by_maxssau"
 				(path "/48e19dd7-3c62-4fd7-8a3b-78a40c79d086/523f9a2f-ddd1-4c6e-b1cf-fbf0997bf88b/7af472cf-3fd2-4e4b-b7f3-feb3f131a7f1"
-					(reference "R200")
+					(reference "R187")
 					(unit 1)
 				)
@@
 		(dnp no)
 		(fields_autoplaced yes)
-		(property "Reference" "R194"
+		(property "Reference" "R181"
 			(at 85.09 132.08 90)
 			(effects
@@
 			(project "kharon386mod_by_maxssau"
 				(path "/48e19dd7-3c62-4fd7-8a3b-78a40c79d086/523f9a2f-ddd1-4c6e-b1cf-fbf0997bf88b/7af472cf-3fd2-4e4b-b7f3-feb3f131a7f1"
-					(reference "R194")
+					(reference "R181")
 					(unit 1)
 				)
@@
 		(dnp no)
 		(fields_autoplaced yes)
-		(property "Reference" "R197"
+		(property "Reference" "R184"
 			(at 166.37 102.87 90)
 			(effects
@@
 			(project "kharon386mod_by_maxssau"
 				(path "/48e19dd7-3c62-4fd7-8a3b-78a40c79d086/523f9a2f-ddd1-4c6e-b1cf-fbf0997bf88b/7af472cf-3fd2-4e4b-b7f3-feb3f131a7f1"
-					(reference "R197")
+					(reference "R184")
 					(unit 1)
 				)
@@
 		(dnp no)
 		(fields_autoplaced yes)
-		(property "Reference" "R190"
+		(property "Reference" "R180"
 			(at 82.55 95.25 90)
 			(effects
@@
 			(project "kharon386mod_by_maxssau"
 				(path "/48e19dd7-3c62-4fd7-8a3b-78a40c79d086/523f9a2f-ddd1-4c6e-b1cf-fbf0997bf88b/7af472cf-3fd2-4e4b-b7f3-feb3f131a7f1"
-					(reference "R190")
+					(reference "R180")
 					(unit 1)
 				)
@@
 		(dnp no)
 		(fields_autoplaced yes)
-		(property "Reference" "C206"
+		(property "Reference" "C197"
 			(at 76.2 66.0399 0)
 			(effects
@@
 			(project "kharon386mod_by_maxssau"
 				(path "/48e19dd7-3c62-4fd7-8a3b-78a40c79d086/523f9a2f-ddd1-4c6e-b1cf-fbf0997bf88b/7af472cf-3fd2-4e4b-b7f3-feb3f131a7f1"
-					(reference "C206")
+					(reference "C197")
 					(unit 1)
 				)
@@
 		(dnp no)
 		(fields_autoplaced yes)
-		(property "Reference" "R187"
+		(property "Reference" "R174"
 			(at 39.37 64.77 90)
 			(effects
@@
 			(project "kharon386mod_by_maxssau"
 				(path "/48e19dd7-3c62-4fd7-8a3b-78a40c79d086/523f9a2f-ddd1-4c6e-b1cf-fbf0997bf88b/7af472cf-3fd2-4e4b-b7f3-feb3f131a7f1"
-					(reference "R187")
+					(reference "R174")
 					(unit 1)
 				)
@@
 		(dnp no)
 		(fields_autoplaced yes)
-		(property "Reference" "R189"
+		(property "Reference" "R178"
 			(at 60.96 57.15 90)
 			(effects
@@
 			(project "kharon386mod_by_maxssau"
 				(path "/48e19dd7-3c62-4fd7-8a3b-78a40c79d086/523f9a2f-ddd1-4c6e-b1cf-fbf0997bf88b/7af472cf-3fd2-4e4b-b7f3-feb3f131a7f1"
-					(reference "R189")
+					(reference "R178")
 					(unit 1)
 				)
@@
 		(dnp no)
 		(fields_autoplaced yes)
-		(property "Reference" "C204"
+		(property "Reference" "C195"
 			(at 53.34 66.0399 0)
 			(effects
@@
 			(project "kharon386mod_by_maxssau"
 				(path "/48e19dd7-3c62-4fd7-8a3b-78a40c79d086/523f9a2f-ddd1-4c6e-b1cf-fbf0997bf88b/7af472cf-3fd2-4e4b-b7f3-feb3f131a7f1"
-					(reference "C204")
+					(reference "C195")
 					(unit 1)
 				)
@@
 		(dnp no)
 		(fields_autoplaced yes)
-		(property "Reference" "U41"
+		(property "Reference" "U35"
 			(at 34.29 165.0999 0)
 			(effects
@@
 			(project ""
 				(path "/48e19dd7-3c62-4fd7-8a3b-78a40c79d086/523f9a2f-ddd1-4c6e-b1cf-fbf0997bf88b/7af472cf-3fd2-4e4b-b7f3-feb3f131a7f1"
-					(reference "U41")
+					(reference "U35")
 					(unit 3)
 				)
@@
 		(dnp no)
 		(fields_autoplaced yes)
-		(property "Reference" "L25"
+		(property "Reference" "L24"
 			(at 39.37 58.42 90)
 			(effects
@@
 			(project "kharon386mod_by_maxssau"
 				(path "/48e19dd7-3c62-4fd7-8a3b-78a40c79d086/523f9a2f-ddd1-4c6e-b1cf-fbf0997bf88b/7af472cf-3fd2-4e4b-b7f3-feb3f131a7f1"
-					(reference "L25")
+					(reference "L24")
 					(unit 1)
 				)
@@
 		(dnp no)
 		(fields_autoplaced yes)
-		(property "Reference" "R191"
+		(property "Reference" "R182"
 			(at 114.3 114.3 90)
 			(effects
@@
 			(project "kharon386mod_by_maxssau"
 				(path "/48e19dd7-3c62-4fd7-8a3b-78a40c79d086/523f9a2f-ddd1-4c6e-b1cf-fbf0997bf88b/7af472cf-3fd2-4e4b-b7f3-feb3f131a7f1"
-					(reference "R191")
+					(reference "R182")
 					(unit 1)
 				)
@@
 		(dnp no)
 		(fields_autoplaced yes)
-		(property "Reference" "R199"
+		(property "Reference" "R186"
 			(at 203.2 92.71 90)
 			(effects
@@
 			(project "kharon386mod_by_maxssau"
 				(path "/48e19dd7-3c62-4fd7-8a3b-78a40c79d086/523f9a2f-ddd1-4c6e-b1cf-fbf0997bf88b/7af472cf-3fd2-4e4b-b7f3-feb3f131a7f1"
-					(reference "R199")
+					(reference "R186")
 					(unit 1)
 				)
@@
 		(dnp no)
 		(fields_autoplaced yes)
-		(property "Reference" "R196"
+		(property "Reference" "R183"
 			(at 166.37 92.71 90)
 			(effects
@@
 			(project "kharon386mod_by_maxssau"
 				(path "/48e19dd7-3c62-4fd7-8a3b-78a40c79d086/523f9a2f-ddd1-4c6e-b1cf-fbf0997bf88b/7af472cf-3fd2-4e4b-b7f3-feb3f131a7f1"
-					(reference "R196")
+					(reference "R183")
 					(unit 1)
 				)
@@
 		(dnp no)
 		(fields_autoplaced yes)
-		(property "Reference" "R201"
+		(property "Reference" "R188"
 			(at 234.95 111.76 90)
 			(effects
@@
 			(project "kharon386mod_by_maxssau"
 				(path "/48e19dd7-3c62-4fd7-8a3b-78a40c79d086/523f9a2f-ddd1-4c6e-b1cf-fbf0997bf88b/7af472cf-3fd2-4e4b-b7f3-feb3f131a7f1"
-					(reference "R201")
+					(reference "R188")
 					(unit 1)
 				)
@@
 		(dnp no)
 		(fields_autoplaced yes)
-		(property "Reference" "R192"
+		(property "Reference" "R175"
 			(at 45.72 95.25 90)
 			(effects
@@
 			(project "kharon386mod_by_maxssau"
 				(path "/48e19dd7-3c62-4fd7-8a3b-78a40c79d086/523f9a2f-ddd1-4c6e-b1cf-fbf0997bf88b/7af472cf-3fd2-4e4b-b7f3-feb3f131a7f1"
-					(reference "R192")
+					(reference "R175")
 					(unit 1)
 				)
@@
 		(on_board yes)
 		(dnp no)
-		(property "Reference" "U41"
+		(property "Reference" "U37"
 			(at 86.3601 114.3 90)
 			(effects
@@
 			(project ""
 				(path "/48e19dd7-3c62-4fd7-8a3b-78a40c79d086/523f9a2f-ddd1-4c6e-b1cf-fbf0997bf88b/7af472cf-3fd2-4e4b-b7f3-feb3f131a7f1"
-					(reference "U41")
+					(reference "U37")
 					(unit 1)
 				)
@@
 		(dnp no)
 		(fields_autoplaced yes)
-		(property "Reference" "C205"
+		(property "Reference" "C196"
 			(at 71.12 48.2599 0)
 			(effects
@@
 			(project "kharon386mod_by_maxssau"
 				(path "/48e19dd7-3c62-4fd7-8a3b-78a40c79d086/523f9a2f-ddd1-4c6e-b1cf-fbf0997bf88b/7af472cf-3fd2-4e4b-b7f3-feb3f131a7f1"
-					(reference "C205")
-					(unit 1)
-				)
+					(reference "C196")
+					(unit 1)
+				)
