File: HW/KiCAD/kharon386mod_by_maxssau.kicad_pcb (KiCad board)
At the start: 4 copper layers, 398 parts, among them CON1 CF-CARD-cfcard, IC1 RTL8019AS, J1 USB_A, J10 PC104_16, J11 PC104, J12 USB_B, J13 POWER 5V2A, J14 COM1, J15 COM2, J16 ESP, J17 Mini-DIN-6, J18 Mini-DIN-6, J19 Vol. Btns, J2 IO ADDR1, J20 Conn_02x08_Odd_Even, J21 PJ-320, J22 DB15_Female_HighDensity_Mount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, J23 PJ-320, J3 IO ADDR2, J4 Conn_01x02_Pin, J5 IO-ADDR, J6 CONFIG, J7 CONFIG, J8 RJ45_LED_Shielded, J9 Conn_01x04, Q1 BC817, Q2 BC856, Q3 BC856, SW1 Jumper / Pin header 1x2 Pitch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, SW2 SW_Push, SW3 SW_DIP_x01, SW4 VGA Config, U1 74LS138, U10 74HCT32PW, U11 MSM5118160F-JS, U12 74HCT138PW, U13 ST16C554D, U14 74HCT138PW, U15 GD75232PW, U16 GD75232PW, U17 MAX809LEUR, U18 CH340G, U19 LMR62014, U2 CH375B, U20 ESP-12F, U21 IP4220CZ6, U22 IP4220CZ6, U23 1117-3.3, U24 ICL7660A, U25 39SF040, U26 TXS0104PW, U27 MT4C4256, U28 TVGA9000I, U29 MT4C4256, U3 74LS139, U30 MT4C4256, U31 27C512, U32 MT4C4256, U33 74HCT138PW, U34 93C66A, U35 ES1868F, U36 1117-3.3, U37 1117-5.0, U38 1117-5.0, U39 SAM2695, U4 74LS125, U40 NE5532DR, U5 93LCxxB, U6 MSM5118160F-JS, U7 M6117D, U8 MSM5118160F-JS, U9 MSM5118160F-JS, X1 14.318 MHz, X2 80 MHz, X3 1.8432 Mhz, Y1 12M, Y2 20MHz, Y3 32768 Hz, Y4 12 MHz, Y5 40 MHz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

Commit message: pcb edit
Parts:
- removed RN1, RN2, RN3, RN4: 4.7k, Resistor_SMD:R_Array_Convex_4x0603
- removed RN5, RN6: 330, Resistor_SMD:R_Array_Convex_4x0603
- removed RN7: 1k, Resistor_SMD:R_Array_Convex_4x0603
- added R100: 4.7k, Resistor_SMD:R_0805_2012Metric_Pad1.20x1.40mm_HandSolder, B.Cu at (949.1, -130.8)
- added R101: 4.7k, Resistor_SMD:R_0805_2012Metric_Pad1.20x1.40mm_HandSolder, B.Cu at (949.1, -133.1)
- added R102: 4.7k, Resistor_SMD:R_0805_2012Metric_Pad1.20x1.40mm_HandSolder, B.Cu at (949.1, -135.4)
- added R103: 4.7k, Resistor_SMD:R_0805_2012Metric_Pad1.20x1.40mm_HandSolder, B.Cu at (954.3, -136.1)
- added R104: 4.7k, Resistor_SMD:R_0805_2012Metric_Pad1.20x1.40mm_HandSolder, B.Cu at (934.1, -144.8)
- added R105: 4.7k, Resistor_SMD:R_0805_2012Metric_Pad1.20x1.40mm_HandSolder, B.Cu at (954.2, -161.3)
- added R106: 4.7k, Resistor_SMD:R_0805_2012Metric_Pad1.20x1.40mm_HandSolder, B.Cu at (954.2, -166.2)
- added R107: 4.7k, Resistor_SMD:R_0805_2012Metric_Pad1.20x1.40mm_HandSolder, B.Cu at (938.3, -135.9)
- added R108: 4.7k, Resistor_SMD:R_0805_2012Metric_Pad1.20x1.40mm_HandSolder, B.Cu at (922.9, -143.6)
- added R109: 4.7k, Resistor_SMD:R_0805_2012Metric_Pad1.20x1.40mm_HandSolder, B.Cu at (938.3, -163.8)
- added R110: 4.7k, Resistor_SMD:R_0805_2012Metric_Pad1.20x1.40mm_HandSolder, B.Cu at (954.3, -181.6)
- added R111: 4.7k, Resistor_SMD:R_0805_2012Metric_Pad1.20x1.40mm_HandSolder, B.Cu at (954.3, -143.5)
- added R112: 4.7k, Resistor_SMD:R_0805_2012Metric_Pad1.20x1.40mm_HandSolder, B.Cu at (938.3, -143.5)
- added R113: 4.7k, Resistor_SMD:R_0805_2012Metric_Pad1.20x1.40mm_HandSolder, B.Cu at (938.3, -146.1)
- added R114: 4.7k, Resistor_SMD:R_0805_2012Metric_Pad1.20x1.40mm_HandSolder, B.Cu at (938.3, -148.6)
- added R115: 4.7k, Resistor_SMD:R_0805_2012Metric_Pad1.20x1.40mm_HandSolder, B.Cu at (938.3, -151.1)
- added R116: 4.7k, Resistor_SMD:R_0805_2012Metric_Pad1.20x1.40mm_HandSolder, B.Cu at (954.3, -141.0)
- added R117: 4.7k, Resistor_SMD:R_0805_2012Metric_Pad1.20x1.40mm_HandSolder, B.Cu at (954.3, -179.1)
- added R88: 4.7k, Resistor_SMD:R_0805_2012Metric_Pad1.20x1.40mm_HandSolder, B.Cu at (938.3, -184.2)
- added R93: 4.7k, Resistor_SMD:R_0805_2012Metric_Pad1.20x1.40mm_HandSolder, B.Cu at (954.2, -158.8)
- added R94: 4.7k, Resistor_SMD:R_0805_2012Metric_Pad1.20x1.40mm_HandSolder, B.Cu at (938.3, -158.8)
- added R95: 4.7k, Resistor_SMD:R_0805_2012Metric_Pad1.20x1.40mm_HandSolder, B.Cu at (954.2, -163.8)
- added R96: 4.7k, Resistor_SMD:R_0805_2012Metric_Pad1.20x1.40mm_HandSolder, B.Cu at (949.1, -121.3)
- added R97: 4.7k, Resistor_SMD:R_0805_2012Metric_Pad1.20x1.40mm_HandSolder, B.Cu at (949.1, -123.2)
- added R98: 4.7k, Resistor_SMD:R_0805_2012Metric_Pad1.20x1.40mm_HandSolder, B.Cu at (949.1, -125.7)
- added R99: 4.7k, Resistor_SMD:R_0805_2012Metric_Pad1.20x1.40mm_HandSolder, B.Cu at (949.1, -128.3)
- C100, C101, C104, C105, C106, C107, C108, C109, C110, C111, C112, C113, C114, C115, C117, C118, C119, C120, C121, C123, C124, C125, C126, C127, C128, C129, C131, C132, C133, C134, C137, C139, C144, C145, C146, C147, C148, C151, C152, C155, C157, C158, C159, C160, C161, C162, C163, C164, C165, C166, C167, C168, C169, C170, C171, C172, C173, C174, C175, C176, C177, C178, C29, C30, C31, C33, C34, C35, C36, C37, C38, C39, C40, C41, C42, C43, C44, C45, C46, C47, C48, C49, C50, C51, C52, C53, C54, C55, C56, C57, C58, C59, C60, C61, C62, C63, C64, C65, C66, C67, C68, C69, C71, C73, C76, C77, C79, C80, C81, C82, C83, C85, C86, C87, C88, C90, C91, C92, C96, C97, C99: footprint Capacitor_SMD:C_0603_1608Metric_Pad1.08x0.95mm_HandSolder -> Capacitor_SMD:C_0805_2012Metric_Pad1.18x1.45mm_HandSolder
- L3: moved to B.Cu
- L4: footprint Inductor_SMD:L_Taiyo-Yuden_NR-60xx_HandSoldering -> Inductor_SMD:L_Panasonic_PCC-M0850M
- R24, R25, R27: footprint Resistor_SMD:R_0603_1608Metric_Pad0.98x0.95mm_HandSolder -> Resistor_SMD:R_0805_2012Metric_Pad1.20x1.40mm_HandSolder; moved to B.Cu
- R26, R28, R29, R31, R32, R33, R34, R35, R36, R37, R38, R39, R40, R43, R44, R45, R46, R47, R48, R49, R50, R51, R52, R53, R54, R55, R56, R57, R58, R59, R60, R61, R62, R63, R64, R65, R66, R67, R68, R69, R70, R71, R72, R73, R74, R75, R76, R77, R78, R79, R80, R82, R83, R86, R87, R89, R90, R91, R92: footprint Resistor_SMD:R_0603_1608Metric_Pad0.98x0.95mm_HandSolder -> Resistor_SMD:R_0805_2012Metric_Pad1.20x1.40mm_HandSolder
- moved SW3 1241.5 mm to (1133.1, -217.7)
- moved R32 994.7 mm to (938.3, -191.8), turned to 180 degrees
- moved J11 968.3 mm to (942.3, -118.1), turned to 180 degrees
- moved L3 952.9 mm to (937.6, -123.2)
- moved J10 948.8 mm to (947.4, -138.4), turned to 180 degrees
- moved R24 932.7 mm to (901.6, -154.2), turned to 180 degrees
- moved U11 930.1 mm to (885.2, -151.9)
- moved U6 930.1 mm to (843.2, -151.9)
- moved U8 930.1 mm to (857.2, -151.9)
- moved U9 930.1 mm to (871.2, -151.9)
- moved C52 930.1 mm to (878.3, -137.7)
- moved C55 930.1 mm to (864.3, -137.7)
- moved C58 930.1 mm to (850.3, -137.6)
- moved C61 930.1 mm to (839.1, -137.6)
- moved R26 925.5 mm to (906.5, -129.0)
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Routing:
- net GND: vias 0 -> 1
- net /B_ISA_IOCHK: vias 0 -> 1
- net (no net): vias 0 -> 2

Commit message: some eidts, remove com
Parts:
- removed the J13 at (828.8, -14.5)
- removed J21, J23: PJ-320, Library_user:PJ-320A_D
- removed J22: DB15_Female_HighDensity_MountingHoles, Library_user:DSUB-15-HD_Female_Horizontal_P2.29x1.98mm_EdgePinOffset3.03mm_Housed_MountingHolesOffset4.94mm
- removed U38: 1117-5.0, Package_TO_SOT_SMD:SOT-223-3_TabPin2
- removed U39: SAM2695, Package_DFN_QFN:QFN-48-1EP_6x6mm_P0.4mm_EP4.2x4.2mm
- removed U40: NE5532DR, Package_SO:SOIC-8_3.9x4.9mm_P1.27mm
- removed X3: 1.8432 Mhz, Oscillator:Oscillator_SMD_Abracon_ASV-4Pin_7.0x5.1mm_HandSoldering
- removed Y6: 12 MHz, Crystal:Crystal_SMD_SeikoEpson_TSX3225-4Pin_3.2x2.5mm_HandSoldering
- added C179: 100n, Capacitor_SMD:C_0805_2012Metric_Pad1.18x1.45mm_HandSolder, F.Cu at (872.9, 157.7)
- added C180: 1u, Capacitor_THT:C_Rect_L7.0mm_W2.5mm_P5.00mm, F.Cu at (872.2, 161.2)
- added C181: 1u, Capacitor_THT:C_Rect_L7.0mm_W2.5mm_P5.00mm, F.Cu at (872.2, 165.3)
- added C182: 100n, Capacitor_SMD:C_0805_2012Metric_Pad1.18x1.45mm_HandSolder, F.Cu at (847.5, 177.4)
- added C183: 100n, Capacitor_SMD:C_0805_2012Metric_Pad1.18x1.45mm_HandSolder, F.Cu at (847.5, 180.4)
- added C184: 100n, Capacitor_SMD:C_0805_2012Metric_Pad1.18x1.45mm_HandSolder, F.Cu at (847.5, 183.4)
- added C185: 100n, Capacitor_SMD:C_0805_2012Metric_Pad1.18x1.45mm_HandSolder, F.Cu at (847.5, 186.4)
- added C186: 1u, Capacitor_THT:C_Rect_L7.0mm_W2.5mm_P5.00mm, F.Cu at (846.8, 190.0)
- added C187: 1u, Capacitor_THT:C_Rect_L7.0mm_W2.5mm_P5.00mm, F.Cu at (846.8, 194.0)
- added C188: 100n, Capacitor_SMD:C_0805_2012Metric_Pad1.18x1.45mm_HandSolder, F.Cu at (847.5, 148.7)
- added C189: 100n, Capacitor_SMD:C_0805_2012Metric_Pad1.18x1.45mm_HandSolder, F.Cu at (847.5, 151.7)
- added C190: 100n, Capacitor_SMD:C_0805_2012Metric_Pad1.18x1.45mm_HandSolder, F.Cu at (847.5, 154.7)
- added C191: 100n, Capacitor_SMD:C_0805_2012Metric_Pad1.18x1.45mm_HandSolder, F.Cu at (847.5, 157.7)
- added C192: 1u, Capacitor_THT:C_Rect_L7.0mm_W2.5mm_P5.00mm, F.Cu at (846.8, 161.2)
- added C193: 1u, Capacitor_THT:C_Rect_L7.0mm_W2.5mm_P5.00mm, F.Cu at (846.8, 165.3)
- added C194: 100n, Capacitor_SMD:C_0805_2012Metric_Pad1.18x1.45mm_HandSolder, F.Cu at (872.9, 177.4)
- added C195: 100n, Capacitor_SMD:C_0805_2012Metric_Pad1.18x1.45mm_HandSolder, F.Cu at (872.9, 180.4)
- added C196: 100n, Capacitor_SMD:C_0805_2012Metric_Pad1.18x1.45mm_HandSolder, F.Cu at (872.9, 183.4)
- added C197: 100n, Capacitor_SMD:C_0805_2012Metric_Pad1.18x1.45mm_HandSolder, F.Cu at (872.9, 186.4)
- added J11: Mini-DIN-6, Library_user:minidin-6, F.Cu at (919.5, -215.9)
- added JP2: OpenIn, Jumper:SolderJumper-2_P1.3mm_Open_TrianglePad1.0x1.5mm, F.Cu at (855.8, 219.6)
- added JP3: OpenOut, Jumper:SolderJumper-2_P1.3mm_Open_TrianglePad1.0x1.5mm, F.Cu at (855.8, 223.1)
- added JP4: OpenIn, Jumper:SolderJumper-2_P1.3mm_Open_TrianglePad1.0x1.5mm, F.Cu at (877.4, 149.0)
- added JP5: OpenOut, Jumper:SolderJumper-2_P1.3mm_Open_TrianglePad1.0x1.5mm, F.Cu at (877.4, 152.5)
- added JP6: OpenIn, Jumper:SolderJumper-2_P1.3mm_Open_TrianglePad1.0x1.5mm, F.Cu at (852.0, 177.7)
- added JP7: OpenOut, Jumper:SolderJumper-2_P1.3mm_Open_TrianglePad1.0x1.5mm, F.Cu at (852.0, 181.2)
- added JP8: OpenIn, Jumper:SolderJumper-2_P1.3mm_Open_TrianglePad1.0x1.5mm, F.Cu at (852.0, 149.0)
- added JP9: OpenOut, Jumper:SolderJumper-2_P1.3mm_Open_TrianglePad1.0x1.5mm, F.Cu at (852.0, 152.5)
- added L16: BLM21, Inductor_SMD:L_0805_2012Metric_Pad1.15x1.40mm_HandSolder, F.Cu at (833.2, 209.0)
- added L17: BLM21, Inductor_SMD:L_0805_2012Metric_Pad1.15x1.40mm_HandSolder, F.Cu at (858.6, 148.7)
- added L18: BLM21, Inductor_SMD:L_0805_2012Metric_Pad1.15x1.40mm_HandSolder, F.Cu at (858.6, 151.6)
- added L19: BLM21, Inductor_SMD:L_0805_2012Metric_Pad1.15x1.40mm_HandSolder, F.Cu at (833.2, 177.4)
- added L20: BLM21, Inductor_SMD:L_0805_2012Metric_Pad1.15x1.40mm_HandSolder, F.Cu at (833.2, 180.3)
- added L21: BLM21, Inductor_SMD:L_0805_2012Metric_Pad1.15x1.40mm_HandSolder, F.Cu at (833.2, 148.7)
- added L22: BLM21, Inductor_SMD:L_0805_2012Metric_Pad1.15x1.40mm_HandSolder, F.Cu at (833.2, 151.6)
- added L23: BLM21, Inductor_SMD:L_0805_2012Metric_Pad1.15x1.40mm_HandSolder, F.Cu at (858.6, 177.4)
- added L24: BLM21, Inductor_SMD:L_0805_2012Metric_Pad1.15x1.40mm_HandSolder, F.Cu at (858.6, 180.3)
- added R118: 10k, Resistor_SMD:R_0805_2012Metric_Pad1.20x1.40mm_HandSolder, F.Cu at (842.7, 209.0)
- added R119: 3k, Resistor_SMD:R_0805_2012Metric_Pad1.20x1.40mm_HandSolder, F.Cu at (842.7, 212.0)
- added R120: 1n, Resistor_SMD:R_0805_2012Metric_Pad1.20x1.40mm_HandSolder, F.Cu at (842.7, 214.9)
- added R121: 100, Resistor_SMD:R_0805_2012Metric_Pad1.20x1.40mm_HandSolder, F.Cu at (842.7, 217.9)
- added R122: 10, Resistor_SMD:R_0805_2012Metric_Pad1.20x1.40mm_HandSolder, F.Cu at (858.6, 154.6)
- added R123: 10, Resistor_SMD:R_0805_2012Metric_Pad1.20x1.40mm_HandSolder, F.Cu at (858.6, 157.5)
- added R124: 10, Resistor_SMD:R_0805_2012Metric_Pad1.20x1.40mm_HandSolder, F.Cu at (858.6, 160.5)
- added R125: 10, Resistor_SMD:R_0805_2012Metric_Pad1.20x1.40mm_HandSolder, F.Cu at (858.6, 163.4)
- added R126: 4.7k, Resistor_SMD:R_0805_2012Metric_Pad1.20x1.40mm_HandSolder, F.Cu at (858.6, 166.4)
- added R127: 10k, Resistor_SMD:R_0805_2012Metric_Pad1.20x1.40mm_HandSolder, F.Cu at (863.3, 148.7)
- added R128: 3k, Resistor_SMD:R_0805_2012Metric_Pad1.20x1.40mm_HandSolder, F.Cu at (863.3, 151.6)
- added R129: 10k, Resistor_SMD:R_0805_2012Metric_Pad1.20x1.40mm_HandSolder, F.Cu at (863.3, 154.6)
- added R130: 4.7k, Resistor_SMD:R_0805_2012Metric_Pad1.20x1.40mm_HandSolder, F.Cu at (863.3, 157.5)
- added R131: 1n, Resistor_SMD:R_0805_2012Metric_Pad1.20x1.40mm_HandSolder, F.Cu at (863.3, 160.5)
- added R132: 3k, Resistor_SMD:R_0805_2012Metric_Pad1.20x1.40mm_HandSolder, F.Cu at (863.3, 163.4)
- added R133: 10k, Resistor_SMD:R_0805_2012Metric_Pad1.20x1.40mm_HandSolder, F.Cu at (863.3, 166.4)
- added R134: 1.6k, Resistor_SMD:R_0805_2012Metric_Pad1.20x1.40mm_HandSolder, F.Cu at (868.1, 148.7)
- added R135: 10k, Resistor_SMD:R_0805_2012Metric_Pad1.20x1.40mm_HandSolder, F.Cu at (868.1, 151.6)
- added R136: 3k, Resistor_SMD:R_0805_2012Metric_Pad1.20x1.40mm_HandSolder, F.Cu at (868.1, 154.6)
- added R137: 1n, Resistor_SMD:R_0805_2012Metric_Pad1.20x1.40mm_HandSolder, F.Cu at (868.1, 157.5)
- added R138: 100, Resistor_SMD:R_0805_2012Metric_Pad1.20x1.40mm_HandSolder, F.Cu at (868.1, 160.5)
- added R139: 10, Resistor_SMD:R_0805_2012Metric_Pad1.20x1.40mm_HandSolder, F.Cu at (833.2, 183.3)
- added R140: 10, Resistor_SMD:R_0805_2012Metric_Pad1.20x1.40mm_HandSolder, F.Cu at (833.2, 186.2)
- added R141: 10, Resistor_SMD:R_0805_2012Metric_Pad1.20x1.40mm_HandSolder, F.Cu at (833.2, 189.2)
- added R142: 10, Resistor_SMD:R_0805_2012Metric_Pad1.20x1.40mm_HandSolder, F.Cu at (833.2, 192.1)
- added R143: 4.7k, Resistor_SMD:R_0805_2012Metric_Pad1.20x1.40mm_HandSolder, F.Cu at (833.2, 195.1)
- added R144: 10k, Resistor_SMD:R_0805_2012Metric_Pad1.20x1.40mm_HandSolder, F.Cu at (837.9, 177.4)
- added R145: 3k, Resistor_SMD:R_0805_2012Metric_Pad1.20x1.40mm_HandSolder, F.Cu at (837.9, 180.3)
- added R146: 10k, Resistor_SMD:R_0805_2012Metric_Pad1.20x1.40mm_HandSolder, F.Cu at (837.9, 183.3)
- added R147: 4.7k, Resistor_SMD:R_0805_2012Metric_Pad1.20x1.40mm_HandSolder, F.Cu at (837.9, 186.2)
- added R148: 1n, Resistor_SMD:R_0805_2012Metric_Pad1.20x1.40mm_HandSolder, F.Cu at (837.9, 189.2)
- added R149: 3k, Resistor_SMD:R_0805_2012Metric_Pad1.20x1.40mm_HandSolder, F.Cu at (837.9, 192.1)
- added R150: 10k, Resistor_SMD:R_0805_2012Metric_Pad1.20x1.40mm_HandSolder, F.Cu at (837.9, 195.1)
- added R151: 1.6k, Resistor_SMD:R_0805_2012Metric_Pad1.20x1.40mm_HandSolder, F.Cu at (842.7, 177.4)
- added R152: 10k, Resistor_SMD:R_0805_2012Metric_Pad1.20x1.40mm_HandSolder, F.Cu at (842.7, 180.3)
- added R153: 3k, Resistor_SMD:R_0805_2012Metric_Pad1.20x1.40mm_HandSolder, F.Cu at (842.7, 183.3)
- added R154: 1n, Resistor_SMD:R_0805_2012Metric_Pad1.20x1.40mm_HandSolder, F.Cu at (842.7, 186.2)
- added R155: 100, Resistor_SMD:R_0805_2012Metric_Pad1.20x1.40mm_HandSolder, F.Cu at (842.7, 189.2)
- added R156: 10, Resistor_SMD:R_0805_2012Metric_Pad1.20x1.40mm_HandSolder, F.Cu at (833.2, 154.6)
- added R157: 10, Resistor_SMD:R_0805_2012Metric_Pad1.20x1.40mm_HandSolder, F.Cu at (833.2, 157.5)
- added R158: 10, Resistor_SMD:R_0805_2012Metric_Pad1.20x1.40mm_HandSolder, F.Cu at (833.2, 160.5)
- added R159: 10, Resistor_SMD:R_0805_2012Metric_Pad1.20x1.40mm_HandSolder, F.Cu at (833.2, 163.4)
- added R160: 4.7k, Resistor_SMD:R_0805_2012Metric_Pad1.20x1.40mm_HandSolder, F.Cu at (833.2, 166.4)
- added R161: 10k, Resistor_SMD:R_0805_2012Metric_Pad1.20x1.40mm_HandSolder, F.Cu at (837.9, 148.7)
- added R162: 3k, Resistor_SMD:R_0805_2012Metric_Pad1.20x1.40mm_HandSolder, F.Cu at (837.9, 151.6)
- added R163: 10k, Resistor_SMD:R_0805_2012Metric_Pad1.20x1.40mm_HandSolder, F.Cu at (837.9, 154.6)
- added R164: 4.7k, Resistor_SMD:R_0805_2012Metric_Pad1.20x1.40mm_HandSolder, F.Cu at (837.9, 157.5)
- added R165: 1n, Resistor_SMD:R_0805_2012Metric_Pad1.20x1.40mm_HandSolder, F.Cu at (837.9, 160.5)
- added R166: 3k, Resistor_SMD:R_0805_2012Metric_Pad1.20x1.40mm_HandSolder, F.Cu at (837.9, 163.4)
- added R167: 10k, Resistor_SMD:R_0805_2012Metric_Pad1.20x1.40mm_HandSolder, F.Cu at (837.9, 166.4)
- added R168: 1.6k, Resistor_SMD:R_0805_2012Metric_Pad1.20x1.40mm_HandSolder, F.Cu at (842.7, 148.7)
- added R169: 10k, Resistor_SMD:R_0805_2012Metric_Pad1.20x1.40mm_HandSolder, F.Cu at (842.7, 151.6)
- added R170: 3k, Resistor_SMD:R_0805_2012Metric_Pad1.20x1.40mm_HandSolder, F.Cu at (842.7, 154.6)
- added R171: 1n, Resistor_SMD:R_0805_2012Metric_Pad1.20x1.40mm_HandSolder, F.Cu at (842.7, 157.5)
- added R172: 100, Resistor_SMD:R_0805_2012Metric_Pad1.20x1.40mm_HandSolder, F.Cu at (842.7, 160.5)
- added R173: 10, Resistor_SMD:R_0805_2012Metric_Pad1.20x1.40mm_HandSolder, F.Cu at (858.6, 183.3)
- added R174: 10, Resistor_SMD:R_0805_2012Metric_Pad1.20x1.40mm_HandSolder, F.Cu at (858.6, 186.2)
- added R175: 10k, Resistor_SMD:R_0805_2012Metric_Pad1.20x1.40mm_HandSolder, F.Cu at (858.6, 189.2)
- added R176: 10k, Resistor_SMD:R_0805_2012Metric_Pad1.20x1.40mm_HandSolder, F.Cu at (858.6, 192.1)
- added R177: 10, Resistor_SMD:R_0805_2012Metric_Pad1.20x1.40mm_HandSolder, F.Cu at (858.6, 195.1)
- added R178: 10, Resistor_SMD:R_0805_2012Metric_Pad1.20x1.40mm_HandSolder, F.Cu at (863.3, 177.4)
- added R179: 10k, Resistor_SMD:R_0805_2012Metric_Pad1.20x1.40mm_HandSolder, F.Cu at (863.3, 180.3)
- added R180: 10k, Resistor_SMD:R_0805_2012Metric_Pad1.20x1.40mm_HandSolder, F.Cu at (863.3, 183.3)
- added R181: 10k, Resistor_SMD:R_0805_2012Metric_Pad1.20x1.40mm_HandSolder, F.Cu at (863.3, 186.2)
- added R182: 100, Resistor_SMD:R_0805_2012Metric_Pad1.20x1.40mm_HandSolder, F.Cu at (863.3, 189.2)
- added R183: 10k, Resistor_SMD:R_0805_2012Metric_Pad1.20x1.40mm_HandSolder, F.Cu at (863.3, 192.1)
- added R184: 10k, Resistor_SMD:R_0805_2012Metric_Pad1.20x1.40mm_HandSolder, F.Cu at (863.3, 195.1)
- added R185: 10k, Resistor_SMD:R_0805_2012Metric_Pad1.20x1.40mm_HandSolder, F.Cu at (868.1, 177.4)
- added R186: 10k, Resistor_SMD:R_0805_2012Metric_Pad1.20x1.40mm_HandSolder, F.Cu at (868.1, 180.3)
- added R187: 10k, Resistor_SMD:R_0805_2012Metric_Pad1.20x1.40mm_HandSolder, F.Cu at (868.1, 183.3)
- added R188: 100, Resistor_SMD:R_0805_2012Metric_Pad1.20x1.40mm_HandSolder, F.Cu at (868.1, 186.2)
- added RV1: SB, Potentiometer_THT:Potentiometer_Alps_RK163_Dual_Horizontal, F.Cu at (1023.2, -99.1)
- added RV2: MIDI, Potentiometer_THT:Potentiometer_Alps_RK163_Dual_Horizontal, F.Cu at (1042.7, -99.1)
- C100, C99: value 47p -> 10u; footprint Capacitor_SMD:C_0805_2012Metric_Pad1.18x1.45mm_HandSolder -> Capacitor_Tantalum_SMD:CP_EIA-3528-21_Kemet-B_Pad1.50x2.35mm_HandSolder
- C101, C109, C36, C37, C42: value 100n -> 47p
- C102: value 10u -> 47p; footprint Capacitor_Tantalum_SMD:CP_EIA-3528-21_Kemet-B_HandSolder -> Capacitor_SMD:C_0805_2012Metric_Pad1.18x1.45mm_HandSolder
- C103, C135, C136: value 10u -> 100n; footprint Capacitor_Tantalum_SMD:CP_EIA-3528-21_Kemet-B_HandSolder -> Capacitor_SMD:C_0805_2012Metric_Pad1.18x1.45mm_HandSolder
- C104: value 47p -> 100p
- C107: value 100p -> 47p
- C112: value 47p -> 1u
- C113, C114: value 47p -> 100n
- C115: value 1u -> 100u; footprint Capacitor_SMD:C_0805_2012Metric_Pad1.18x1.45mm_HandSolder -> Capacitor_Tantalum_SMD:CP_EIA-7343-31_Kemet-D_Pad2.25x2.55mm_HandSolder
- C116, C123, C157, C158, C40, C45, C48, C51, C54, C57, C60, C63, C66, C68: value 100n -> 1u
- C118, C120, C121, C125, C126: value 220n -> 100n
- C119: value 220n -> 1u
- C122: value 47u/6.3V -> 100n; footprint Capacitor_Tantalum_SMD:CP_EIA-3528-21_Kemet-B_HandSolder -> Capacitor_SMD:C_0805_2012Metric_Pad1.18x1.45mm_HandSolder
- C127: value 4.7n -> 1u
- C128, C129: value 1n -> 100n
- C130, C138, C70, C72, C74, C78: value 10u -> 100n
- C131, C132, C133, C134, C167, C38, C44, C47, C50, C53, C56, C59, C62, C64: value 1u -> 100n
- C137: value 470p -> 100n
- C139: value 10n -> 220n
- C140, C141, C142: value 10u -> 220n; footprint Capacitor_Tantalum_SMD:CP_EIA-3528-21_Kemet-B_HandSolder -> Capacitor_SMD:C_0805_2012Metric_Pad1.18x1.45mm_HandSolder
- C143: value 100u/16V -> 47u/6.3V; footprint Capacitor_Tantalum_SMD:CP_EIA-7343-31_Kemet-D_HandSolder -> Capacitor_Tantalum_SMD:CP_EIA-3528-21_Kemet-B_Pad1.50x2.35mm_HandSolder
- C146, C147: value 100n -> 220n
- C148: value 100n -> 4.7n
- C149, C150: value 10u -> 1n
- C151, C152, C91: value 22p -> 100n
- C153, C154: value 47u -> 10u; footprint Capacitor_Tantalum_SMD:CP_EIA-3528-21_Kemet-B_HandSolder -> Capacitor_SMD:C_0805_2012Metric_Pad1.18x1.45mm_HandSolder
- C155: value 1u -> 22p
- C156: value 100u -> 22p; footprint Capacitor_Tantalum_SMD:CP_EIA-7343-31_Kemet-D_HandSolder -> Capacitor_SMD:C_0805_2012Metric_Pad1.18x1.45mm_HandSolder
- C159, C161, C162, C163, C169: value 100n -> 10u; footprint Capacitor_SMD:C_0805_2012Metric_Pad1.18x1.45mm_HandSolder -> Capacitor_Tantalum_SMD:CP_EIA-3528-21_Kemet-B_Pad1.50x2.35mm_HandSolder
- C160: value 1u -> 470p
- C164: value 1u -> 100u/16V; footprint Capacitor_SMD:C_0805_2012Metric_Pad1.18x1.45mm_HandSolder -> Capacitor_Tantalum_SMD:CP_EIA-7343-31_Kemet-D_Pad2.25x2.55mm_HandSolder
- C165, C77, C79, C82: value 100n -> 10u
- C174, C175: value 100n -> 1u; footprint Capacitor_SMD:C_0805_2012Metric_Pad1.18x1.45mm_HandSolder -> Capacitor_THT:C_Rect_L7.0mm_W2.5mm_P5.00mm
- C41: value 1u -> 47p
- C75: value 220u -> 10u; footprint Capacitor_Tantalum_SMD:CP_EIA-7343-31_Kemet-D_HandSolder -> Capacitor_SMD:C_0805_2012Metric_Pad1.18x1.45mm_HandSolder
- C84: value 2.2u -> 100n
- C88: value 22p -> 2.2u
- C90: value 10n -> 100n
- C96: value 47p -> 220u; footprint Capacitor_SMD:C_0805_2012Metric_Pad1.18x1.45mm_HandSolder -> Capacitor_Tantalum_SMD:CP_EIA-7343-31_Kemet-D_Pad2.25x2.55mm_HandSolder
- C97: value 47p -> 47u; footprint Capacitor_SMD:C_0805_2012Metric_Pad1.18x1.45mm_HandSolder -> Capacitor_Tantalum_SMD:CP_EIA-7343-31_Kemet-D_Pad2.25x2.55mm_HandSolder
- C98: value 47u -> 100n; footprint Capacitor_Tantalum_SMD:CP_EIA-3528-21_Kemet-B_HandSolder -> Capacitor_SMD:C_0805_2012Metric_Pad1.18x1.45mm_HandSolder
- CON1: footprint Library:TE_1734451-1 -> Library_user:TE_1734451-1-LONG
- D4: value BZV55C5V6 -> MBR0520; footprint Diode_SMD:D_MiniMELF -> Diode_SMD:D_SOD-123
- D5: value BT168GW -> MBR0520; footprint Package_TO_SOT_SMD:SOT-223-3_TabPin2 -> Diode_SMD:D_SOD-123
- D7: value MBR0520 -> BZV55C5V6; footprint Diode_SMD:D_SOD-123 -> Diode_SMD:D_MiniMELF
- D8: value MBR0520 -> BT168GW; footprint Diode_SMD:D_SOD-123 -> Package_TO_SOT_SMD:SOT-223-3_TabPin2
- IC1: footprint Library:RTL8019AS -> kharon:RTL8019AS
- J12: value USB_B -> Mini-DIN-6; footprint Connector_USB:USB_B_Lumberg_2411_02_Horizontal -> Library_user:minidin-6
- J14: value COM1 -> USB_B; footprint Connector_PinHeader_2.54mm:PinHeader_2x05_P2.54mm_Vertical -> Connector_USB:USB_B_Lumberg_2411_02_Horizontal
- J15: value COM2 -> POWER 5V2A; footprint Connector_PinHeader_2.54mm:PinHeader_2x05_P2.54mm_Vertical -> TerminalBlock:TerminalBlock_bornier-2_P5.08mm
- J16: value ESP -> Vol. Btns; footprint Connector_PinHeader_2.54mm:PinHeader_2x05_P2.54mm_Vertical -> Connector_PinHeader_2.54mm:PinHeader_2x03_P2.54mm_Vertical
- J17: value Mini-DIN-6 -> PJ-320; footprint Library_user:minidin-6 -> Library_user:PJ-320A_D
- J18: value Mini-DIN-6 -> Conn_02x08_Odd_Even; footprint Library_user:minidin-6 -> Connector_PinSocket_2.54mm:PinSocket_2x08_P2.54mm_Vertical
- J19: value Vol. Btns -> PJ-320; footprint Connector_PinHeader_2.54mm:PinHeader_2x03_P2.54mm_Vertical -> Library_user:PJ-320A_D
- J20: value Conn_02x08_Odd_Even -> DB15_Female_HighDensity_MountingHoles; footprint Connector_PinSocket_2.54mm:PinSocket_2x08_P2.54mm_Vertical -> Library_user:DSUB-15-HD_Female_Horizontal_P2.29x1.98mm_EdgePinOffset3.03mm_Housed_MountingHolesOffset4.94mm
- L10, L11: value 5.6u -> BLM21PG331BH1D; footprint Inductor_SMD:L_1210_3225Metric_Pad1.42x2.65mm_HandSolder -> Inductor_SMD:L_0805_2012Metric_Pad1.15x1.40mm_HandSolder
- L14: value BLM21PG331BH1D -> 5.6u; footprint Inductor_SMD:L_0805_2012Metric_Pad1.15x1.40mm_HandSolder -> Inductor_SMD:L_1210_3225Metric_Pad1.42x2.65mm_HandSolder
- L15: value BLM21PG331BH1D -> BLM21
- L3, R109, R113, R24, R25, R88, R98: moved to F.Cu
- L4: footprint Inductor_SMD:L_Panasonic_PCC-M0850M -> Inductor_SMD:L_7.3x7.3_H4.5
- R100, R101, R99: value 4.7k -> 47k; moved to F.Cu
- R102, R110, R112, R116, R97: value 4.7k -> 10k; moved to F.Cu
- R103, R93, R94, R95: value 4.7k -> 1k; moved to F.Cu
- R104: value 4.7k -> 0; moved to F.Cu
- R105, R106, R107, R108: value 4.7k -> 10; moved to F.Cu
- R111, R115: value 4.7k -> 3k; moved to F.Cu
- R114: value 4.7k -> 1n; moved to F.Cu
- R117: value 4.7k -> 1.6k; moved to F.Cu
- R26, R41, R42: value 22 -> 4.7k
- R27: value 22 -> 4.7k; moved to F.Cu
- R28: value 10M -> 4.7k
- R29, R37, R47: value 1k -> 4.7k
- R30: value 33 -> 22
- R31: value 5.6k -> 22
- R32: value 22 -> 10M
- R33: value 1M -> 4.7k
- R34, R35, R36: value 470 -> 4.7k
- R38, R40, R45, R46, R48, R62, R86, R87, R89, R90: value 10k -> 4.7k
- R39: value 51k -> 4.7k
- R43: value 117k -> 4.7k
- R44: value 13.3k -> 4.7k
- R53, R54: value 33 -> 4.7k
- R55: value 33 -> 1k
- R56: value 150 -> 33
- R57: value 100 -> 10k
- R58: value 150 -> 5.6k
- R59: value 4.7k -> 10k
- R60: value 150 -> 10k
- R61: value 150 -> 4.7k
- R65: value 4.7k -> 22
- R66, R67, R68: value 4.7k -> 470
- R69: value 4.7k -> 51k
- R70: value 10k -> 117k
- R71: value 1k -> 13.3k
- R72: value 1k -> 1M
- R74: value 0 -> 1k
- R76, R77: value 10k -> 33
- R78: value 4.7k -> 150
- R79: value 47k -> 100
- R80: value 1k -> 150
- R81, R85: value 0 -> 4.7k
- R82, R83: value 10k -> 150
- R84: value 0 -> 10k
- R91: value 47k -> 4.7k
- R92: value 47k -> 10k
- R96: value 4.7k -> 33; moved to F.Cu
- SW1: value Jumper / Pin header 1x2 Pitch=2.54mm -> SW_Push; footprint Connector_Molex:Molex_KK-254_AE-6410-02A_1x02_P2.54mm_Vertical -> Button_Switch_THT:SW_Tactile_SPST_Angled_PTS645Vx83-2LFS
- SW2: value SW_Push -> SW_DIP_x01; footprint Button_Switch_THT:SW_Tactile_SPST_Angled_PTS645Vx83-2LFS -> Button_Switch_THT:SW_DIP_SPSTx01_Slide_6.7x4.1mm_W7.62mm_P2.54mm_LowProfile
- SW3: value SW_DIP_x01 -> Jumper / Pin header 1x2 Pitch=2.54mm; footprint Button_Switch_THT:SW_DIP_SPSTx01_Slide_6.7x4.1mm_W7.62mm_P2.54mm_LowProfile -> Connector_Molex:Molex_KK-254_AE-6410-02A_1x02_P2.54mm_Vertical
- U11: value MSM5118160F-JS -> MAX809LEUR; footprint Library_user:SOJ-42 -> Package_TO_SOT_SMD:SOT-23
- U12: value 74HCT138PW -> MSM5118160F-JS; footprint Package_SO:TSSOP-16_4.4x5mm_P0.65mm -> Library_user:SOJ-42
- U13: value ST16C554D -> IP4220CZ6; footprint Package_QFP:LQFP-64_10x10mm_P0.5mm -> Package_SO:TSOP-6_1.65x3.05mm_P0.95mm
- U14: value 74HCT138PW -> IP4220CZ6; footprint Package_SO:TSSOP-16_4.4x5mm_P0.65mm -> Package_SO:TSOP-6_1.65x3.05mm_P0.95mm
- U15: value GD75232PW -> 39SF040; footprint Package_SO:TSSOP-20_4.4x6.5mm_P0.65mm -> Library_user:PLCC-32_11.4x14.0mm_P1.27mm-longpads
- U16: value GD75232PW -> LMR62014; footprint Package_SO:TSSOP-20_4.4x6.5mm_P0.65mm -> Package_TO_SOT_SMD:SOT-23-5_HandSoldering
- U17: value MAX809LEUR -> 1117-3.3; footprint Package_TO_SOT_SMD:SOT-23 -> Package_TO_SOT_SMD:SOT-223-3_TabPin2
- U18: value CH340G -> ICL7660A; footprint Package_SO:SOIC-16_3.9x9.9mm_P1.27mm -> Package_SO:SOIC-8_3.9x4.9mm_P1.27mm
- U19: value LMR62014 -> MT4C4256; footprint Package_TO_SOT_SMD:SOT-23-5_HandSoldering -> Package_DIP:DIP-20_W7.62mm
- U2: footprint Library:SOP28-LL -> kharon:SOP28-LL
- U20: value ESP-12F -> TVGA9000I; footprint RF_Module:ESP-12E -> Package_QFP:PQFP-160_28x28mm_P0.65mm
- U21, U22: value IP4220CZ6 -> MT4C4256; footprint Package_SO:TSOP-6_1.65x3.05mm_P0.95mm -> Package_DIP:DIP-20_W7.62mm
- U23: value 1117-3.3 -> 27C512; footprint Package_TO_SOT_SMD:SOT-223-3_TabPin2 -> Library_user:PLCC-32_11.4x14.0mm_P1.27mm-longpads
- U24: value ICL7660A -> MT4C4256; footprint Package_SO:SOIC-8_3.9x4.9mm_P1.27mm -> Package_DIP:DIP-20_W7.62mm
- U25: value 39SF040 -> 74HCT138PW; footprint Library_user:PLCC-32_11.4x14.0mm_P1.27mm-longpads -> Package_SO:TSSOP-16_4.4x5mm_P0.65mm
- U26: value TXS0104PW -> 93C66A; footprint Package_SO:TSSOP-14_4.4x5mm_P0.65mm -> Package_SO:SOIC-8_3.9x4.9mm_P1.27mm
- U27: value MT4C4256 -> ES1868F; footprint Package_DIP:DIP-20_W7.62mm -> Package_QFP:PQFP-100_14x20mm_P0.65mm
- U28: value TVGA9000I -> SAM2695; footprint Package_QFP:PQFP-160_28x28mm_P0.65mm -> Package_DFN_QFN:QFN-48-1EP_6x6mm_P0.4mm_EP4.2x4.2mm
- U29, U30: value MT4C4256 -> 1117-5.0; footprint Package_DIP:DIP-20_W7.62mm -> Package_TO_SOT_SMD:SOT-223-3_TabPin2
- U31: value 27C512 -> 1117-3.3; footprint Library_user:PLCC-32_11.4x14.0mm_P1.27mm-longpads -> Package_TO_SOT_SMD:SOT-223-3_TabPin2
- U32: value MT4C4256 -> NE5532; footprint Package_DIP:DIP-20_W7.62mm -> Package_SO:SOIC-8_3.9x4.9mm_P1.27mm
- U33: value 74HCT138PW -> NE5532; footprint Package_SO:TSSOP-16_4.4x5mm_P0.65mm -> Package_SO:SOIC-8_3.9x4.9mm_P1.27mm
- U34: value 93C66A -> NE5532
- U35: value ES1868F -> NE5532; footprint Package_QFP:PQFP-100_14x20mm_P0.65mm -> Package_SO:SOIC-8_3.9x4.9mm_P1.27mm
- U36: value 1117-3.3 -> NE5532; footprint Package_TO_SOT_SMD:SOT-223-3_TabPin2 -> Package_SO:SOIC-8_3.9x4.9mm_P1.27mm
- U37: value 1117-5.0 -> NE5532; footprint Package_TO_SOT_SMD:SOT-223-3_TabPin2 -> Package_SO:SOIC-8_3.9x4.9mm_P1.27mm
- Y4: value 12 MHz -> 40 MHz
- Y5: value 40 MHz -> 12 MHz
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- renumbered J11 to J13
Connections:
- C100 pad 1: /ISA_386SX_BOARD/MSCLK -> GND
- C100 pad 2: GND -> -5V
- C101 pad 1: +BATT -> GND
- C101 pad 2: GND -> /ISA_VGA_SB/~{CAS}
- C102 pad 1: Net-(U24-CAP+) -> GND
- C102 pad 2: Net-(U24-CAP-) -> /ISA_VGA_SB/~{RAS}
- C103 pad 1: GND -> Net-(U20-VLF)
- C103 pad 2: -5V -> /ISA_VGA_SB/AVDD1
- C104 pad 1: GND -> Net-(U20-~{IOW})
- C104 pad 2: /ISA_VGA_SB/~{CAS} -> GND
- C105 pad 1: GND -> /B_ISA_SMEMR
- C105 pad 2: /ISA_VGA_SB/~{RAS} -> GND
- C106 pad 1: Net-(U28-VLF) -> GND
- C106 pad 2: /ISA_VGA_SB/AVDD1 -> Net-(C106-Pad2)
- C107 pad 1: Net-(U28-~{IOW}) -> /ISA_VGA_SB/VGA_R
- C108 pad 1: /B_ISA_SMEMR -> /ISA_VGA_SB/VGA_VS
- C109 pad 1: GND -> /ISA_VGA_SB/VGA_G
- C109 pad 2: Net-(C109-Pad2) -> GND
- C110 pad 1: /ISA_VGA_SB/VGA_R -> /ISA_VGA_SB/VGA_HS
- C111 pad 1: /ISA_VGA_SB/VGA_VS -> /ISA_VGA_SB/VGA_B
- C112 pad 1: /ISA_VGA_SB/VGA_G -> /ISA_VGA_SB/VGA_MON
- C113 pad 1: /ISA_VGA_SB/VGA_HS -> +5V
- C114 pad 1: /ISA_VGA_SB/VGA_B -> +5V
- C115 pad 1: /ISA_VGA_SB/VGA_MON -> +5V
- C116 pad 1: /B_ISA_5V0 -> GND
- C116 pad 2: GND -> +3V3
- C117 pad 1: Net-(U35-AUXA_L) -> +5V
- C117 pad 2: Net-(C117-Pad2) -> GND
- C118 pad 1: Net-(U35-AUXB_L) -> +5V
- C118 pad 2: /ISA_VGA_SB/MIDI_L -> GND
- C119 pad 1: Net-(U35-AUXB_R) -> +5V
- C119 pad 2: /ISA_VGA_SB/MIDI_R -> GND
- C120 pad 1: Net-(U35-LINE_L) -> GND
- C120 pad 2: Net-(C120-Pad2) -> +3V3
- C121 pad 1: Net-(U35-LINE_R) -> +5V
- C121 pad 2: Net-(C121-Pad2) -> GND
- C122 pad 1: Net-(U35-CMR) -> +5V
- C123 pad 1: Net-(U35-CMR) -> +5V
- C124 pad 1: Net-(U35-VREF) -> GND
- C124 pad 2: GND -> +3V3
- C125 pad 1: Net-(U35-FOUT_L) -> +5V
- C125 pad 2: Net-(U35-CIN_L) -> GND
- C126 pad 1: Net-(U35-FOUT_R) -> +5V
- C126 pad 2: Net-(U35-CIN_R) -> GND
- C127 pad 1: GND -> +5V
- C127 pad 2: Net-(C117-Pad2) -> GND
- C128 pad 1: Net-(U35-CIN_L) -> +5V
- C129 pad 1: Net-(U35-CIN_R) -> +5V
- C130 pad 1: GND -> +5V
- C130 pad 2: +5V -> GND
- C131 pad 1: +12V -> +5V
- C132 pad 1: +12V -> +5V
- C133 pad 1: Net-(U35-AOUT_R) -> +5V
- C133 pad 2: Net-(C133-Pad2) -> GND
- C134 pad 1: Net-(U35-AOUT_L) -> /B_ISA_5V0
- C134 pad 2: Net-(C134-Pad2) -> GND
- C135 pad 1: Net-(U37-VO) -> +5V
- C136 pad 1: +3V3 -> +5V
- C137 pad 1: /ISA_VGA_SB/RESET -> +5V
- C138 pad 1: GND -> Net-(U27-AUXA_L)
- C138 pad 2: Net-(U40A-+) -> Net-(C138-Pad2)
- C139 pad 1: GND -> Net-(U27-AUXB_L)
- C139 pad 2: Net-(U40A-+) -> /ISA_VGA_SB/MIDI_L
- C140 pad 1: /ISA_VGA_SB/AVDD1 -> Net-(U27-AUXB_R)
- C140 pad 2: GND -> /ISA_VGA_SB/MIDI_R
- C141 pad 1: /ISA_VGA_SB/AVDD2 -> Net-(U27-LINE_L)
- C141 pad 2: GND -> Net-(C141-Pad2)
- C142 pad 1: /ISA_VGA_SB/AVDD_ES -> Net-(U27-LINE_R)
- C142 pad 2: GND -> Net-(C142-Pad2)
- C143 pad 1: /ISA_VGA_SB/AVDD_OP -> Net-(U27-CMR)
- C144 pad 1: GND -> Net-(U27-CMR)
- C144 pad 2: Net-(U39-VCM) -> GND
- C145 pad 1: GND -> Net-(U27-VREF)
- C145 pad 2: Net-(U39-OUTVC12) -> GND
- C146 pad 1: /ISA_VGA_SB/AVDD2 -> Net-(U27-FOUT_L)
- C146 pad 2: GND -> Net-(U27-CIN_L)
- C147 pad 1: /ISA_VGA_SB/AVDD_ES -> Net-(U27-FOUT_R)
- C147 pad 2: GND -> Net-(U27-CIN_R)
- C148 pad 1: /ISA_VGA_SB/AVDD_OP -> GND
- C148 pad 2: GND -> Net-(C138-Pad2)
- C149 pad 1: GND -> Net-(U27-CIN_L)
- C149 pad 2: Net-(U39-OUTVC12) -> GND
- C150 pad 1: GND -> Net-(U27-CIN_R)
- C150 pad 2: Net-(U39-VCM) -> GND
- C151 pad 2: Net-(U39-X2) -> Net-(U28-VCM)
- C152 pad 2: Net-(U39-X1) -> Net-(U28-OUTVC12)
- C153 pad 1: Net-(C153-Pad1) -> GND
- C153 pad 2: Net-(C153-Pad2) -> Net-(U28-OUTVC12)
- C154 pad 1: Net-(C154-Pad1) -> GND
- C154 pad 2: Net-(C154-Pad2) -> Net-(U28-VCM)
- C155 pad 2: +3V3 -> Net-(U28-X2)
- C156 pad 1: +5V -> GND
- C156 pad 2: GND -> Net-(U28-X1)
- C157 pad 1: +5V -> +12V
- C158 pad 1: +5V -> +12V
- C159 pad 1: GND -> Net-(U29-VO)
- C159 pad 2: +3V3 -> GND
- C160 pad 1: +5V -> /ISA_VGA_SB/RESET
- C161 pad 1: +5V -> /ISA_VGA_SB/AVDD1
- C162 pad 1: +5V -> /ISA_VGA_SB/AVDD2
- C163 pad 1: GND -> /ISA_VGA_SB/AVDD_ES
- C163 pad 2: +3V3 -> GND
- C164 pad 1: +5V -> /ISA_VGA_SB/AVDD_OP
- C165 pad 1: +5V -> GND
- C165 pad 2: GND -> +5V
- C166 pad 1: +5V -> /ISA_VGA_SB/AVDD2
- C167 pad 1: +5V -> /ISA_VGA_SB/AVDD_ES
- C168 pad 1: +5V -> /ISA_VGA_SB/AVDD_OP
- C169 pad 1: +5V -> +3V3
- C170 pad 1: +5V -> Net-(C170-Pad1)
- C171 pad 1: +5V -> Net-(C171-Pad1)
- C172 pad 1: +5V -> /ISA_VGA_SB/LPF/LPF_V+
- C173 pad 1: +5V -> /ISA_VGA_SB/LPF/LPF_V-
- C174 pad 1: +5V -> /ISA_VGA_SB/LPF/LPF_AIN
- C174 pad 2: GND -> Net-(JP2-B)
- C175 pad 1: +5V -> Net-(JP3-A)
- C175 pad 2: GND -> Net-(JP3-B)
- C176 pad 1: +5V -> Net-(C176-Pad1)
- C177 pad 1: +5V -> Net-(C177-Pad1)
- C178 pad 1: +5V -> /ISA_VGA_SB/LPF1/LPF_V+
- C32 pad 1: /B_ISA_5V0 -> Net-(Q2-C)
- C36 pad 1: GND -> /ISA_386SX_BOARD/KBDAT
- C36 pad 2: +5V -> GND
- C37 pad 1: GND -> /ISA_386SX_BOARD/MSDAT
- C37 pad 2: +5V -> GND
- C41 pad 1: GND -> /ISA_386SX_BOARD/KBCLK
- C41 pad 2: +5V -> GND
- C42 pad 1: GND -> /ISA_386SX_BOARD/MSCLK
- C42 pad 2: +5V -> GND
- C43 pad 1: +5V -> GND
- C43 pad 2: GND -> +5V
- C46 pad 1: +5V -> GND
- C46 pad 2: GND -> +5V
- C47 pad 1: GND -> +5V
- C47 pad 2: +5V -> GND
- C49 pad 1: +5V -> GND
- C49 pad 2: GND -> +5V
- C50 pad 1: GND -> +5V
- C50 pad 2: +5V -> GND
- C52 pad 1: +5V -> GND
- C52 pad 2: GND -> +5V
- C55 pad 1: +5V -> GND
- C55 pad 2: GND -> +5V
- C57 pad 1: GND -> +5V
- C57 pad 2: +5V -> GND
- C58 pad 1: +5V -> GND
- C58 pad 2: GND -> +5V
- C60 pad 1: GND -> +5V
- C60 pad 2: +5V -> GND
- C61 pad 1: +5V -> GND
- C61 pad 2: GND -> +5V
- C63 pad 1: GND -> +5V
- C63 pad 2: +5V -> GND
- C64 pad 1: +5V -> GND
- C64 pad 2: GND -> +5V
- C65 pad 1: GND -> +5V
- C65 pad 2: +5V -> GND
- C66 pad 1: GND -> +5V
- C66 pad 2: +5V -> GND
- C67 pad 2: +12V -> +5V
- C68 pad 1: GND -> +5V
- C68 pad 2: +5V -> GND
- C69 pad 2: +12V -> +5V
- C70 pad 1: +5V -> GND
- C70 pad 2: GND -> +5V
- C71 pad 1: GND -> /B_ISA_5V0
- C71 pad 2: +5V -> GND
- C72 pad 1: +5V -> GND
- C72 pad 2: GND -> +12V
- C74 pad 1: +5V -> GND
- C74 pad 2: GND -> +12V
- C76 pad 2: -12V -> +5V
- C77 pad 1: GND -> +5V
- C77 pad 2: +5V -> GND
- C78 pad 1: +5V -> GND
- C78 pad 2: GND -> +5V
- C79 pad 1: GND -> +5V
- C79 pad 2: -12V -> GND
- C80 pad 2: +5V -> -12V
- C82 pad 1: GND -> +5V
- C82 pad 2: +5V -> GND
- C83 pad 2: +3V3 -> -12V
- C86 pad 2: +3V3 -> +5V
- C87 pad 1: Net-(Q3-C) -> GND
- C87 pad 2: GND -> +3V3
- C88 pad 1: Net-(U18-XO) -> GND
- C88 pad 2: GND -> +5V
- C89 pad 1: Net-(D7-A) -> GND
- C89 pad 2: Net-(D6-A) -> +5V
- C90 pad 2: Net-(U18-V3) -> +3V3
- C91 pad 1: Net-(U18-XI) -> Net-(D5-A)
- C91 pad 2: GND -> Net-(D4-A)
- C92 pad 2: Net-(U19-FB) -> Net-(U16-FB)
- C96 pad 1: /ISA_386SX_BOARD/KBDAT -> +5V
- C97 pad 1: /ISA_386SX_BOARD/MSDAT -> +3V3
- C98 pad 1: +3V3 -> +BATT
- C99 pad 1: /ISA_386SX_BOARD/KBCLK -> Net-(U18-CAP+)
- C99 pad 2: GND -> Net-(U18-CAP-)
- D4 pad 1: +5V -> GND
- D5 pad 1: GND -> +12V
- D5 pad 2: +5V -> Net-(D5-A)
- D6 pad 1: GND -> Net-(D4-A)
- D6 pad 2: Net-(D6-A) -> -12V
- D7 pad 1: +12V -> +5V
- D8 pad 1: Net-(D6-A) -> GND
- D8 pad 2: -12V -> +5V
- F1 pad 2: Net-(SW1-B) -> Net-(SW3-B)
- J12 pad 1: unconnected-(J12-VBUS-Pad1) -> /ISA_386SX_BOARD/MSDAT
- J12 pad 2: /ISA_386SX_BOARD/USB_DN -> unconnected-(J12-Pad2)
- J12 pad 3: /ISA_386SX_BOARD/USB_DP -> GND
- J12 pad 4: GND -> +5V
- J12 pad 5: Net-(J12-Shield) -> /ISA_386SX_BOARD/MSCLK
- J13 pad 59: Net-(J11-Pin_59) -> Net-(J13-Pin_59)
- J14 pad 1: /ISA_386SX_BOARD/DCD1 -> unconnected-(J14-VBUS-Pad1)
- J14 pad 2: /ISA_386SX_BOARD/RX1 -> /ISA_386SX_BOARD/USB_DN
- J14 pad 3: /ISA_386SX_BOARD/TX1 -> /ISA_386SX_BOARD/USB_DP
- J14 pad 4: /ISA_386SX_BOARD/DTR1 -> GND
- J14 pad 5: GND -> Net-(J14-Shield)
- J15 pad 1: /ISA_386SX_BOARD/DCD2 -> Net-(J15-Pin_1)
- J15 pad 2: /ISA_386SX_BOARD/RX2 -> GND
- J16 pad 1: /ISA_386SX_BOARD/ESP_BOOT -> GND
- J16 pad 2: GND -> Net-(J16-Pin_2)
- J16 pad 3: /ISA_386SX_BOARD/ESP_TX -> GND
- J16 pad 5: /ISA_386SX_BOARD/ESP_RX -> GND
- J18 pad 1: /ISA_386SX_BOARD/MSDAT -> /ISA_VGA_SB/AOUT_L
- J18 pad 2: unconnected-(J18-Pad2) -> /ISA_VGA_SB/AOUT_R
- J18 pad 4: +5V -> GND
- J18 pad 5: /ISA_386SX_BOARD/MSCLK -> /ISA_VGA_SB/VGA_R
- J18 pad 6: unconnected-(J18-Pad6) -> Net-(J18-Pin_6)
- J20 pad 1: /ISA_VGA_SB/AOUT_L -> /ISA_VGA_SB/VGA_R
- J20 pad 10: /ISA_VGA_SB/VGA_HS -> GND
- J20 pad 11: GND -> unconnected-(J20-Pad11)
- J20 pad 12: GND -> /ISA_VGA_SB/VGA_MON
- J20 pad 13: /ISA_VGA_SB/VGA_B -> /ISA_VGA_SB/VGA_HS
- J20 pad 2: /ISA_VGA_SB/AOUT_R -> /ISA_VGA_SB/VGA_G
- J20 pad 3: GND -> /ISA_VGA_SB/VGA_B
- J20 pad 4: GND -> unconnected-(J20-Pad4)
- J20 pad 5: /ISA_VGA_SB/VGA_R -> GND
- J20 pad 6: Net-(J20-Pin_6) -> GND
- J20 pad 8: /ISA_VGA_SB/VGA_MON -> GND
- J20 pad 9: /ISA_VGA_SB/VGA_G -> Net-(J20-Pad9)
- L10 pad 1: +5V -> /ISA_VGA_SB/AnalogSumm2CH/ASUMM_OUTL
- L10 pad 2: /ISA_VGA_SB/AVDD_ES -> /ISA_VGA_SB/AOUT_L
- L11 pad 1: Net-(U37-VO) -> /ISA_VGA_SB/AnalogSumm2CH/ASUMM_OUTR
- L11 pad 2: /ISA_VGA_SB/AVDD1 -> /ISA_VGA_SB/AOUT_R
- L12 pad 1: Net-(U37-VO) -> Net-(U29-VO)
- L12 pad 2: /ISA_VGA_SB/AVDD2 -> /ISA_VGA_SB/AVDD1
- L13 pad 1: Net-(L13-Pad1) -> Net-(U29-VO)
- L13 pad 2: /ISA_VGA_SB/AVDD_OP -> /ISA_VGA_SB/AVDD2
- L14 pad 1: Net-(C153-Pad2) -> +12V
- L14 pad 2: /ISA_VGA_SB/AOUT_R -> /ISA_VGA_SB/AVDD_OP
- L15 pad 1: Net-(C154-Pad2) -> /ISA_VGA_SB/AVDD_OP
- L15 pad 2: /ISA_VGA_SB/AOUT_L -> Net-(C170-Pad1)
- L4 pad 2: Net-(D7-A) -> Net-(D5-A)
- L5 pad 1: Net-(C109-Pad2) -> Net-(C106-Pad2)
- L5 pad 2: Net-(U28-XTL1) -> Net-(U20-XTL1)
- L7 pad 1: Net-(C120-Pad2) -> Net-(C141-Pad2)
- L8 pad 1: Net-(C121-Pad2) -> Net-(C142-Pad2)
- Q2 pad 1: /ISA_386SX_BOARD/ESP_TX -> Net-(Q2-B)
- Q2 pad 2: Net-(Q2-E) -> +5V
- Q2 pad 3: GND -> Net-(Q2-C)
- Q3 pad 1: Net-(Q3-B) -> /ISA_386SX_BOARD/ESP_TX
- Q3 pad 2: +5V -> Net-(Q3-E)
- Q3 pad 3: Net-(Q3-C) -> GND
- R100 pad 1: /B_ISA_D3 -> GND
- R100 pad 2: +5V -> /ISA_VGA_SB/AOUT_R
- R101 pad 1: /B_ISA_D2 -> GND
- R101 pad 2: +5V -> /ISA_VGA_SB/AOUT_L
- R102 pad 1: /B_ISA_D1 -> +5V
- R102 pad 2: +5V -> /B_ISA_MEMCS16
- R103 pad 1: /B_ISA_D0 -> /B_ISA_RSTDRV
- R103 pad 2: +5V -> /ISA_VGA_SB/RESET
- R104 pad 1: /B_ISA_AEN -> +5V
- R104 pad 2: +5V -> Net-(J20-Pad9)
- R105 pad 1: /B_ISA_MEMR -> /ISA_VGA_SB/AVDD_OP
- R105 pad 2: +5V -> Net-(C170-Pad1)
- R106 pad 1: /B_ISA_MEMW -> -12V
- R106 pad 2: +5V -> Net-(C171-Pad1)
- R107 pad 1: /ISA_386SX_BOARD/NOWS -> Net-(C170-Pad1)
- R107 pad 2: +5V -> /ISA_VGA_SB/LPF/LPF_V+
- R108 pad 1: /B_ISA_IORDY -> Net-(C171-Pad1)
- R108 pad 2: +5V -> /ISA_VGA_SB/LPF/LPF_V-
- R109 pad 1: /B_ISA_REFRESH -> Net-(JP2-B)
- R109 pad 2: +5V -> Net-(R109-Pad2)
- R110 pad 1: /ISA_386SX_BOARD/MASTER -> /ISA_VGA_SB/LPF/LPF_V-
- R110 pad 2: +5V -> Net-(U33A-+)
- R111 pad 1: /ISA_386SX_BOARD/IOCS16 -> Net-(R109-Pad2)
- R111 pad 2: +5V -> Net-(U33A--)
- R112 pad 1: /B_ISA_SMEMW -> Net-(U33A-+)
- R112 pad 2: +5V -> /ISA_VGA_SB/LPF/LPF_V+
- R113 pad 1: /B_ISA_SMEMR -> Net-(R109-Pad2)
- R113 pad 2: +5V -> Net-(R113-Pad2)
- R114 pad 1: /B_ISA_IOW -> Net-(U33A--)
- R114 pad 2: +5V -> Net-(R113-Pad2)
- R115 pad 1: /B_ISA_IOR -> Net-(R113-Pad2)
- R115 pad 2: +5V -> Net-(R115-Pad2)
- R116 pad 1: /B_ISA_MEMCS16 -> /ISA_VGA_SB/LPF/LPF_V-
- R116 pad 2: +5V -> Net-(U32B-+)
- R117 pad 1: /B_ISA_IOCHK -> Net-(R115-Pad2)
- R117 pad 2: +5V -> Net-(U32B--)
- R25 pad 2: /ISA_386SX_BOARD/KBSJ -> /B_ISA_TC
- R26 pad 1: Net-(U7-OSC14M) -> GND
- R26 pad 2: /B_ISA_14M -> /B_ISA_DACK0
- R27 pad 1: Net-(U7-BCLK2) -> GND
- R27 pad 2: /ISA_386SX_BOARD/CLK2 -> /B_ISA_DACK1
- R28 pad 1: Net-(U7-XTAL1) -> GND
- R28 pad 2: Net-(U7-XTAL2) -> /B_ISA_DACK5
- R29 pad 1: /ISA_386SX_BOARD/SPKR -> GND
- R29 pad 2: Net-(Q1-B) -> /ISA_386SX_BOARD/KBSJ
- R30 pad 1: Net-(J9-Pin_1) -> Net-(U7-OSC14M)
- R30 pad 2: Net-(Q1-C) -> /B_ISA_14M
- R31 pad 1: Net-(CON1-~{INPACK}) -> Net-(U7-BCLK2)
- R31 pad 2: GND -> /ISA_386SX_BOARD/CLK2
- R32 pad 1: Net-(J11-Pin_59) -> Net-(U7-XTAL1)
- R32 pad 2: /B_ISA_14M -> Net-(U7-XTAL2)
- R33 pad 1: Net-(J12-Shield) -> /B_ISA_D7
- R33 pad 2: GND -> +5V
- R34 pad 1: Net-(D1-K) -> /B_ISA_D6
- R34 pad 2: Net-(Q2-E) -> +5V
- R35 pad 1: Net-(D2-K) -> /B_ISA_D5
- R35 pad 2: /ISA_386SX_BOARD/~{CF_BUSY} -> +5V
- R36 pad 1: Net-(D3-K) -> /B_ISA_D4
- R36 pad 2: GND -> +5V
- R37 pad 1: Net-(D4-A) -> /B_ISA_D3
- R37 pad 2: GND -> +5V
- R38 pad 1: Net-(Q3-B) -> /B_ISA_D2
- R38 pad 2: GND -> +5V
- R39 pad 1: +5V -> /B_ISA_D1
- R39 pad 2: Net-(U19-~{SHDN}) -> +5V
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Routing:
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