File: HW/KiCAD/isa_vga_sb.kicad_sch (KiCad schematic)
At the start: 162 parts, among them J19 Vol. Btns, J20 Conn_02x08_Odd_Even, J21 PJ-320, J22 DB15_Female_HighDensity_Mount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, J23 PJ-320, J24 PC104_16, J25 PC104, J26 ESP, J27 Conn_02x07_Odd_Even, SW4 VGA Config, U27 MT4C4256, U28 TVGA9000I, U29 MT4C4256, U30 MT4C4256, U31 27C512, U32 MT4C4256, U33 74HCT138PW, U34 93C66A, U35 ES1868F, U36 1117-3.3, U37 1117-5.0, U38 1117-5.0, U39 SAM2695, U40 NE5532DR, Y5 40 MHz, Y6 12 MHz

Commit message: some edit
Parts:
- removed C179: 470p, Capacitor_SMD:C_0603_1608Metric_Pad1.08x0.95mm_HandSolder, symbol Device:C
- removed J24: PC104_16, Connector_PinHeader_2.54mm:PinHeader_2x20_P2.54mm_Vertical, symbol Connector_Generic:Conn_02x20_Odd_Even
- removed J25: PC104, Connector_PinHeader_2.54mm:PinHeader_2x32_P2.54mm_Vertical, symbol Connector_Generic:Conn_02x32_Odd_Even
- removed J26: ESP, Connector_PinSocket_2.54mm:PinSocket_2x05_P2.54mm_Vertical, symbol Connector_Generic:Conn_02x05_Odd_Even
- removed J27: Conn_02x07_Odd_Even, Connector_PinHeader_2.54mm:PinHeader_2x08_P2.54mm_Vertical, symbol Connector_Generic:Conn_02x08_Odd_Even
- removed R88: 10k, Resistor_SMD:R_0603_1608Metric_Pad0.98x0.95mm_HandSolder, symbol Device:R
- removed R93: 1k, Resistor_SMD:R_0603_1608Metric_Pad0.98x0.95mm_HandSolder, symbol Device:R
- C122, C153, C154: footprint Capacitor_Tantalum_SMD:CP_EIA-3528-21_Kemet-B_Pad1.50x2.35mm_HandSolder -> Capacitor_Tantalum_SMD:CP_EIA-3528-21_Kemet-B_HandSolder
- C135, C136, C140, C141, C142: footprint Capacitor_Tantalum_SMD:CP_EIA-3216-18_Kemet-A_Pad1.58x1.35mm_HandSolder -> Capacitor_Tantalum_SMD:CP_EIA-3528-21_Kemet-B_HandSolder
- C143: footprint Capacitor_Tantalum_SMD:CP_EIA-6032-28_Kemet-C_Pad2.25x2.35mm_HandSolder -> Capacitor_Tantalum_SMD:CP_EIA-7343-31_Kemet-D_HandSolder
- C156: footprint Capacitor_Tantalum_SMD:CP_EIA-7343-31_Kemet-D_Pad2.25x2.55mm_HandSolder -> Capacitor_Tantalum_SMD:CP_EIA-7343-31_Kemet-D_HandSolder
- J21, J23: footprint my:PJ-320A_D -> Library_user:PJ-320A_D
- J22: footprint Connector_Dsub:DSUB-15-HD_Female_Horizontal_P2.29x1.98mm_EdgePinOffset3.03mm_Housed_MountingHolesOffset4.94mm -> Library_user:DSUB-15-HD_Female_Horizontal_P2.29x1.98mm_EdgePinOffset3.03mm_Housed_MountingHolesOffset4.94mm
- LOGO2: footprint mygraphic:black-mage-12.5x8.6 -> Library_user:black-mage-12.5x8.6
- U28: footprint my:PQFP-160_28x28mm_P0.65mm_LongPads -> Package_QFP:PQFP-160_28x28mm_P0.65mm
- U31: footprint my:PLCC-32_11.4x14.0mm_P1.27mm-longpads -> Library_user:PLCC-32_11.4x14.0mm_P1.27mm-longpads
- U35: footprint my:PQFP-100_14x20mm_P0.65mm_ESxxx -> Package_QFP:PQFP-100_14x20mm_P0.65mm
Connections:
- net SND_L is gone; now on net AOUT_L: J20.1 (Pin_1), J21.T
- net SND_R is gone; now on net AOUT_R: J20.2 (Pin_2), J21.R1
- no-connect marks 96 -> 66
Other:
- note removed: "PC/104"

Commit message: pcb edit
Parts:
- C104, C105, C106, C107, C108, C109, C110, C111, C112, C113, C114, C115, C117, C118, C119, C120, C121, C123, C124, C125, C126, C127, C128, C129, C131, C132, C133, C134, C137, C139, C144, C145, C146, C147, C148, C151, C152, C155, C157, C158, C159, C160, C161, C162, C163, C164, C165, C166, C167, C168, C169, C170, C171, C172, C173, C174, C175, C176, C177, C178: footprint Capacitor_SMD:C_0603_1608Metric_Pad1.08x0.95mm_HandSolder -> Capacitor_SMD:C_0805_2012Metric_Pad1.18x1.45mm_HandSolder
- R53, R54, R55, R56, R57, R58, R59, R60, R61, R62, R63, R64, R65, R66, R67, R68, R69, R70, R71, R72, R73, R74, R75, R76, R77, R78, R79, R80, R82, R83, R86, R87, R89, R90, R91, R92: footprint Resistor_SMD:R_0603_1608Metric_Pad0.98x0.95mm_HandSolder -> Resistor_SMD:R_0805_2012Metric_Pad1.20x1.40mm_HandSolder

Commit message: add LPF
Parts:
- removed C133, C134: 1u, Capacitor_SMD:C_0805_2012Metric_Pad1.18x1.45mm_HandSolder, symbol Device:C
- removed C138: 10u, Capacitor_SMD:C_0805_2012Metric_Pad1.18x1.45mm_HandSolder, symbol Device:C
- removed C139: 10n, Capacitor_SMD:C_0805_2012Metric_Pad1.18x1.45mm_HandSolder, symbol Device:C
- removed C153, C154: 47u, Capacitor_Tantalum_SMD:CP_EIA-3528-21_Kemet-B_HandSolder, symbol Device:C_Polarized
- removed L10: 5.6u, Inductor_SMD:L_1210_3225Metric_Pad1.42x2.65mm_HandSolder, symbol Device:L
- removed L14, L15: BLM21PG331BH1D, Inductor_SMD:L_0805_2012Metric_Pad1.15x1.40mm_HandSolder, symbol Device:L
- removed R81, R84, R85: 0, Resistor_SMD:R_0805_2012Metric_Pad1.20x1.40mm_HandSolder, symbol Device:R
- removed R82, R83, R86, R87, R89, R90: 10k, Resistor_SMD:R_0805_2012Metric_Pad1.20x1.40mm_HandSolder, symbol Device:R
- removed R91, R92: 47k, Resistor_SMD:R_0805_2012Metric_Pad1.20x1.40mm_HandSolder, symbol Device:R
- removed U40: NE5532DR, Package_SO:SOIC-8_3.9x4.9mm_P1.27mm, symbol Amplifier_Operational:NE5532
- added L16, L26: BLM21PG331BH1D, Inductor_SMD:L_0805_2012Metric_Pad1.15x1.40mm_HandSolder, symbol Device:L
- added R118, R202: 47k, Resistor_SMD:R_0805_2012Metric_Pad1.20x1.40mm_HandSolder, symbol Device:R
- added RV1: SB, Potentiometer_THT:Potentiometer_Alps_RK163_Dual_Horizontal, symbol Device:R_Potentiometer_Dual
- added RV2: MIDI, Potentiometer_THT:Potentiometer_Alps_RK163_Dual_Horizontal, symbol Device:R_Potentiometer_Dual
Connections:
- net +12V: now also L13.1
- net AOUT_L: now also L16.2, R118.2
- net AOUT_R: now also L26.2, R202.2
- net GND: now also R118.1, R202.1, RV1.1, RV1.4, RV2.1, RV2.4
- net MIDI_L: no longer U39.1 (AOUTL)
- net MIDI_R: no longer U39.2 (AOUTR)
- net at U35.50 (AOUT_L): now also RV1.3
- net at U35.51 (AOUT_R): now also RV1.6
- new net: RV2.3, U39.2 (AOUTR)
- new net: RV2.6, U39.1 (AOUTL)
- new net AnalogSumm2CH/AOUTL: L16.1
- new net AnalogSumm2CH/AOUTR: L26.1
- new net LPF/AIN: RV2.5
- new net LPF1/AIN: RV2.2
- new net LPF2/AIN: RV1.2
- new net LPF3/AIN: RV1.5
Other:
- added sheet AnalogSumm2CH (AnalogSumm2CH.kicad_sch)
- added sheet LPF (lpf.kicad_sch)
- added sheet LPF1 (lpf.kicad_sch)
- added sheet LPF2 (lpf.kicad_sch)
- added sheet LPF3 (lpf.kicad_sch)
- note removed: "Install R40 or R41 R41 recommended"
- note removed: "Install U1 or R38 R38 recommended"
- note removed: "Install U8 or L10 U8 recommended"
- moved on the sheet: C116, C130, C131, C132, C135, C136, C137, C140, C141, C142, C143, C144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

Commit message: some eidts, remove com
Parts:
- C115: renamed from C156; footprint Capacitor_Tantalum_SMD:CP_EIA-7343-31_Kemet-D_HandSolder -> Capacitor_Tantalum_SMD:CP_EIA-7343-31_Kemet-D_Pad2.25x2.55mm_HandSolder
- C143: renamed from C122; footprint Capacitor_Tantalum_SMD:CP_EIA-3528-21_Kemet-B_HandSolder -> Capacitor_Tantalum_SMD:CP_EIA-3528-21_Kemet-B_Pad1.50x2.35mm_HandSolder
- C159: renamed from C135; footprint Capacitor_Tantalum_SMD:CP_EIA-3528-21_Kemet-B_HandSolder -> Capacitor_Tantalum_SMD:CP_EIA-3528-21_Kemet-B_Pad1.50x2.35mm_HandSolder
- C161: renamed from C140; footprint Capacitor_Tantalum_SMD:CP_EIA-3528-21_Kemet-B_HandSolder -> Capacitor_Tantalum_SMD:CP_EIA-3528-21_Kemet-B_Pad1.50x2.35mm_HandSolder
- C162: renamed from C141; footprint Capacitor_Tantalum_SMD:CP_EIA-3528-21_Kemet-B_HandSolder -> Capacitor_Tantalum_SMD:CP_EIA-3528-21_Kemet-B_Pad1.50x2.35mm_HandSolder
- C163: renamed from C142; footprint Capacitor_Tantalum_SMD:CP_EIA-3528-21_Kemet-B_HandSolder -> Capacitor_Tantalum_SMD:CP_EIA-3528-21_Kemet-B_Pad1.50x2.35mm_HandSolder
- C164: renamed from C143; footprint Capacitor_Tantalum_SMD:CP_EIA-7343-31_Kemet-D_HandSolder -> Capacitor_Tantalum_SMD:CP_EIA-7343-31_Kemet-D_Pad2.25x2.55mm_HandSolder
- C169: renamed from C136; footprint Capacitor_Tantalum_SMD:CP_EIA-3528-21_Kemet-B_HandSolder -> Capacitor_Tantalum_SMD:CP_EIA-3528-21_Kemet-B_Pad1.50x2.35mm_HandSolder
- renumbered C104 to C101, C105 to C102, C106 to C103, C107 to C104, C108 to C105, C109 to C106, C110 to C107, C111 to C108, C112 to C109, C113 to C110, C114 to C111, C115 to C112, C157 to C113, C158 to C114, C155 to C116, C161 to C117, C162 to C118, C160 to C119, C159 to C120, C165 to C121, C166 to C122, C164 to C123, C163 to C124, C168 to C125, C169 to C126, C167 to C127, C170 to C128, C171 to C129, C172 to C130, C173 to C131, C174 to C132, C175 to C133, C116 to C134, C176 to C135, C177 to C136, C178 to C137, C117 to C138, C118 to C139, C119 to C140, C120 to C141, C121 to C142, C123 to C144, C124 to C145, C125 to C146, C126 to C147, C127 to C148, C128 to C149, C129 to C150, C144 to C151, C145 to C152, C149 to C153, C150 to C154, C151 to C155, C152 to C156, C131 to C157, C132 to C158, C137 to C160, C130 to C165, C146 to C166, C147 to C167, C148 to C168, J19 to J16, J23 to J17, J20 to J18, J21 to J19, J22 to J20, L16 to L10, L26 to L11, L11 to L12, L12 to L13, L13 to L14, R202 to R100, R118 to R101, R77 to R102, R80 to R103, R74 to R104, R53 to R75, R54 to R76, R55 to R77, R56 to R78, R57 to R79, R58 to R80, R59 to R81, R60 to R82, R61 to R83, R62 to R84, R63 to R85, R64 to R86, R65 to R87, R66 to R88, R67 to R89, R68 to R90, R69 to R91, R70 to R92, R71 to R93, R72 to R94, R73 to R95, R75 to R96, R76 to R97, R78 to R98, R79 to R99, U27 to U19, U28 to U20, U29 to U21, U30 to U22, U31 to U23, U32 to U24, U33 to U25, U34 to U26, U35 to U27, U39 to U28, U37 to U29, U38 to U30, U36 to U31, Y5 to Y4, Y6 to Y5

Commit message: some edits, add HP amp
Parts:
- removed C165: 10u, Capacitor_SMD:C_0805_2012Metric_Pad1.18x1.45mm_HandSolder, symbol Device:C
- removed C168: 100n, Capacitor_SMD:C_0805_2012Metric_Pad1.18x1.45mm_HandSolder, symbol Device:C
- removed C169: 10u, Capacitor_Tantalum_SMD:CP_EIA-3528-21_Kemet-B_Pad1.50x2.35mm_HandSolder, symbol Device:C_Polarized
- removed J18: Conn_02x08_Odd_Even, Connector_PinSocket_2.54mm:PinSocket_2x08_P2.54mm_Vertical, symbol Connector_Generic:Conn_02x08_Odd_Even
- removed L14: 5.6u, Inductor_SMD:L_1210_3225Metric_Pad1.42x2.65mm_HandSolder, symbol Device:L
- removed LOGO2: graphic, Library_user:black-mage-12.5x8.6, symbol my:logo
- removed U31: 1117-3.3, Package_TO_SOT_SMD:SOT-223-3_TabPin2, symbol Regulator_Linear:AMS1117-3.3
- added C165: 10u, Capacitor_Tantalum_SMD:CP_EIA-3528-21_Kemet-B_Pad1.50x2.35mm_HandSolder, symbol Device:C_Polarized
- added J21: PJ-320, Library_user:PJ-320A_D, symbol Connector_Audio:AudioJack4
- added L30, L31: BLM21, Inductor_SMD:L_0805_2012Metric_Pad1.15x1.40mm_HandSolder, symbol Device:L
- added R204, R205: 10, Resistor_SMD:R_0805_2012Metric_Pad1.20x1.40mm_HandSolder, symbol Device:R
- C164: value 100u/16V -> 10u; footprint Capacitor_Tantalum_SMD:CP_EIA-7343-31_Kemet-D_Pad2.25x2.55mm_HandSolder -> Capacitor_Tantalum_SMD:CP_EIA-3528-21_Kemet-B_Pad1.50x2.35mm_HandSolder
Connections:
- net AVDD_OP is gone; now on net AVDD_ES: C164.1
- net +3V3: now also L30.1, R204.1; no longer U28.6 (VA33)
- net AVDD_ES: now also L31.2, R205.2; no longer C163.1, C167.1, U30.2 (VO)
- net GND: now also J19.S, C165.2, J21.R2, J21.S
- new net: C163.1, C167.1, L31.1, R205.1, U30.2 (VO)
- new net: C165.1, L30.2, R204.2, U28.6 (VA33)
- new net HP_OUT_L: J21.T
- new net HP_OUT_R: J21.R1
- no-connect marks 66 -> 65
Other:
- added sheet HPAmp (HPAmp.kicad_sch)
- note removed: "VGA & Sound"
- moved on the sheet: C107, C108, C109, C110, C111, C112, C151, C152, C153, C154, C155, C156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
